File: designs/automatic lights/schm1.brd (EAGLE design)
At the start: 160 x 100 mm, 36 parts, among them IC1 PIC18F4550_40, IC2 7805T, T1 2N3904, T2 2N3904, T3 2N3904, T4 2N3904, T5 2N3904, T6 2N3904, T7 2N3904, T8 2N3904

Commit message: Cambios en tarjeta PCB
Connections:
- removed net N$1: IC1.1
- removed net N$10: IC1.10
- removed net N$17: IC1.17
- removed net N$8: IC1.8
- removed net N$9: IC1.9
- removed net RA3: IC1.5, R9.1
- removed net RA4: IC1.6, R10.1
- removed net RA5: IC1.7, R11.1
- removed net RA6: IC1.14, R12.1
- removed net RC0: IC1.15, R15.1
- removed net RC1: IC1.16, R17.1
- new net N1: IC1.18
- new net OUT1: IC1.8, R9.1
- new net OUT2: IC1.7, R10.1
- new net OUT3: IC1.6, R11.1
- new net OUT4: IC1.5, R12.1
- new net OUT5: IC1.4, R13.1
- new net OUT6: IC1.3, R14.1
- new net OUT7: IC1.2, R15.1
- new net OUT8: IC1.1, R17.1
- new net T_O: IC1.16, SV2.3
- new net T_OF: IC1.17, SV2.1
- net CLK: now also IC1.15; no longer IC1.3
- net DAT: now also IC1.14; no longer IC1.4
- net RB6: no longer R13.1
- net RB7: no longer R14.1
- net RC6: no longer SV2.3
- net RC7: no longer SV2.1
- net RST: now also IC1.10; no longer IC1.2
- net VCC: now also IC1.9
Routing:
- net OUT8: track 0.00 -> 106.2 mm
- net OUT7: track 0.00 -> 95.1 mm
- net OUT6: track 0.00 -> 84.8 mm
- net OUT5: track 0.00 -> 74.4 mm
- net RC1: track 67.3 -> 0.00 mm
- net OUT4: track 0.00 -> 66.2 mm
- net OUT3: track 0.00 -> 57.4 mm
- net RC0: track 57.1 -> 0.00 mm
- net VCC: track 213.9 -> 267.1 mm
- net RB7: track 48.5 -> 0.00 mm
- net OUT2: track 0.00 -> 48.5 mm
- net RB6: track 39.9 -> 0.00 mm
- net OUT1: track 0.00 -> 39.6 mm
- net RA6: track 32.8 -> 0.00 mm
- net T_O: track 0.00 -> 31.8 mm
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