File: designs/automatic lights/schm1.sch (EAGLE design)
At the start: 36 parts, among them IC1 PIC18F4550_40, IC2 7805T, T1 2N3904, T2 2N3904, T3 2N3904, T4 2N3904, T5 2N3904, T6 2N3904, T7 2N3904, T8 2N3904

Commit message: Add files via upload
Connections:
- removed net N$35: IC1.RC7/RX/DT/SDO
- removed net N$36: IC1.RC6/TX/CK
- net RC6: now also IC1.RC6/TX/CK
- net RC7: now also IC1.RC7/RX/DT/SDO
Changed lines of the file:
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@@
 <?xml version="1.0" encoding="utf-8"?>
 <!DOCTYPE eagle SYSTEM "eagle.dtd">
-<eagle version="7.6.0">
+<eagle version="6.6.0">
 <drawing>
 <settings>
@@
 <setting verticaltext="up"/>
 </settings>
-<grid distance="50" unitdist="mil" unit="mil" style="lines" multiple="1" display="no" altdistance="0.01" altunitdist="inch" altunit="inch"/>
+<grid distance="0.1" unitdist="inch" unit="inch" style="lines" multiple="1" display="no" altdistance="0.01" altunitdist="inch" altunit="inch"/>
 <layers>
-<layer number="1" name="Top" color="4" fill="1" visible="yes" active="no"/>
-<layer number="2" name="Route2" color="1" fill="3" visible="yes" active="no"/>
-<layer number="3" name="Route3" color="4" fill="3" visible="yes" active="no"/>
-<layer number="4" name="Route4" color="1" fill="4" visible="yes" active="no"/>
-<layer number="5" name="Route5" color="4" fill="4" visible="yes" active="no"/>
-<layer number="6" name="Route6" color="1" fill="8" visible="yes" active="no"/>
-<layer number="7" name="Route7" color="4" fill="8" visible="yes" active="no"/>
-<layer number="8" name="Route8" color="1" fill="2" visible="yes" active="no"/>
-<layer number="9" name="Route9" color="4" fill="2" visible="yes" active="no"/>
-<layer number="10" name="Route10" color="1" fill="7" visible="yes" active="no"/>
-<layer number="11" name="Route11" color="4" fill="7" visible="yes" active="no"/>
-<layer number="12" name="Route12" color="1" fill="5" visible="yes" active="no"/>
-<layer number="13" name="Route13" color="4" fill="5" visible="yes" active="no"/>
-<layer number="14" name="Route14" color="1" fill="6" visible="yes" active="no"/>
-<layer number="15" name="Route15" color="4" fill="6" visible="yes" active="no"/>
-<layer number="16" name="Bottom" color="1" fill="1" visible="yes" active="no"/>
-<layer number="17" name="Pads" color="2" fill="1" visible="yes" active="no"/>
-<layer number="18" name="Vias" color="2" fill="1" visible="yes" active="no"/>
-<layer number="19" name="Unrouted" color="6" fill="1" visible="yes" active="no"/>
-<layer number="20" name="Dimension" color="15" fill="1" visible="yes" active="no"/>
-<layer number="21" name="tPlace" color="7" fill="1" visible="yes" active="no"/>
-<layer number="22" name="bPlace" color="7" fill="1" visible="yes" active="no"/>
-<layer number="23" name="tOrigins" color="15" fill="1" visible="yes" active="no"/>
-<layer number="24" name="bOrigins" color="15" fill="1" visible="yes" active="no"/>
-<layer number="25" name="tNames" color="7" fill="1" visible="yes" active="no"/>
-<layer number="26" name="bNames" color="7" fill="1" visible="yes" active="no"/>
-<layer number="27" name="tValues" color="7" fill="1" visible="yes" active="no"/>
-<layer number="28" name="bValues" color="7" fill="1" visible="yes" active="no"/>
+<layer number="1" name="Top" color="4" fill="1" visible="no" active="no"/>
+<layer number="2" name="Route2" color="1" fill="3" visible="no" active="no"/>
+<layer number="3" name="Route3" color="4" fill="3" visible="no" active="no"/>
+<layer number="4" name="Route4" color="1" fill="4" visible="no" active="no"/>
+<layer number="5" name="Route5" color="4" fill="4" visible="no" active="no"/>
+<layer number="6" name="Route6" color="1" fill="8" visible="no" active="no"/>
+<layer number="7" name="Route7" color="4" fill="8" visible="no" active="no"/>
+<layer number="8" name="Route8" color="1" fill="2" visible="no" active="no"/>
+<layer number="9" name="Route9" color="4" fill="2" visible="no" active="no"/>
+<layer number="10" name="Route10" color="1" fill="7" visible="no" active="no"/>
+<layer number="11" name="Route11" color="4" fill="7" visible="no" active="no"/>
+<layer number="12" name="Route12" color="1" fill="5" visible="no" active="no"/>
+<layer number="13" name="Route13" color="4" fill="5" visible="no" active="no"/>
+<layer number="14" name="Route14" color="1" fill="6" visible="no" active="no"/>
+<layer number="15" name="Route15" color="4" fill="6" visible="no" active="no"/>
+<layer number="16" name="Bottom" color="1" fill="1" visible="no" active="no"/>
+<layer number="17" name="Pads" color="2" fill="1" visible="no" active="no"/>
+<layer number="18" name="Vias" color="2" fill="1" visible="no" active="no"/>
+<layer number="19" name="Unrouted" color="6" fill="1" visible="no" active="no"/>
+<layer number="20" name="Dimension" color="15" fill="1" visible="no" active="no"/>
+<layer number="21" name="tPlace" color="7" fill="1" visible="no" active="no"/>
+<layer number="22" name="bPlace" color="7" fill="1" visible="no" active="no"/>
+<layer number="23" name="tOrigins" color="15" fill="1" visible="no" active="no"/>
+<layer number="24" name="bOrigins" color="15" fill="1" visible="no" active="no"/>
+<layer number="25" name="tNames" color="7" fill="1" visible="no" active="no"/>
+<layer number="26" name="bNames" color="7" fill="1" visible="no" active="no"/>
+<layer number="27" name="tValues" color="7" fill="1" visible="no" active="no"/>
+<layer number="28" name="bValues" color="7" fill="1" visible="no" active="no"/>
 <layer number="29" name="tStop" color="7" fill="3" visible="no" active="no"/>
 <layer number="30" name="bStop" color="7" fill="6" visible="no" active="no"/>
@@
 <layer number="35" name="tGlue" color="7" fill="4" visible="no" active="no"/>
 <layer number="36" name="bGlue" color="7" fill="5" visible="no" active="no"/>
-<layer number="37" name="tTest" color="7" fill="1" visible="yes" active="no"/>
-<layer number="38" name="bTest" color="7" fill="1" visible="yes" active="no"/>
+<layer number="37" name="tTest" color="7" fill="1" visible="no" active="no"/>
+<layer number="38" name="bTest" color="7" fill="1" visible="no" active="no"/>
 <layer number="39" name="tKeepout" color="4" fill="11" visible="no" active="no"/>
 <layer number="40" name="bKeepout" color="1" fill="11" visible="no" active="no"/>
@@
 <layer number="44" name="Drills" color="7" fill="1" visible="no" active="no"/>
 <layer number="45" name="Holes" color="7" fill="1" visible="no" active="no"/>
-<layer number="46" name="Milling" color="3" fill="1" visible="yes" active="no"/>
-<layer number="47" name="Measures" color="7" fill="1" visible="yes" active="no"/>
-<layer number="48" name="Document" color="7" fill="1" visible="yes" active="no"/>
-<layer number="49" name="Reference" color="7" fill="1" visible="yes" active="no"/>
-<layer number="51" name="tDocu" color="6" fill="1" visible="yes" active="no"/>
-<layer number="52" name="bDocu" color="7" fill="1" visible="yes" active="no"/>
+<layer number="46" name="Milling" color="3" fill="1" visible="no" active="no"/>
+<layer number="47" name="Measures" color="7" fill="1" visible="no" active="no"/>
+<layer number="48" name="Document" color="7" fill="1" visible="no" active="no"/>
+<layer number="49" name="Reference" color="7" fill="1" visible="no" active="no"/>
+<layer number="51" name="tDocu" color="6" fill="1" visible="no" active="no"/>
+<layer number="52" name="bDocu" color="7" fill="1" visible="no" active="no"/>
 <layer number="90" name="Modules" color="5" fill="1" visible="yes" active="yes"/>
 <layer number="91" name="Nets" color="2" fill="1" visible="yes" active="yes"/>
@@
 </segment>
 </net>
-<net name="N$35" class="0">
-<segment>
-<pinref part="IC1" gate="G$1" pin="RC7/RX/DT/SDO"/>
-<wire x1="102.87" y1="59.69" x2="111.76" y2="59.69" width="0.1524" layer="91"/>
-<wire x1="111.76" y1="59.69" x2="111.76" y2="54.61" width="0.1524" layer="91"/>
-<wire x1="111.76" y1="54.61" x2="116.84" y2="54.61" width="0.1524" layer="91"/>
-<label x="116.84" y="54.61" size="1.778" layer="95" xref="yes"/>
-</segment>
-</net>
-<net name="N$36" class="0">
-<segment>
-<pinref part="IC1" gate="G$1" pin="RC6/TX/CK"/>
-<wire x1="102.87" y1="57.15" x2="110.49" y2="57.15" width="0.1524" layer="91"/>
-<wire x1="110.49" y1="57.15" x2="110.49" y2="50.8" width="0.1524" layer="91"/>
-<wire x1="110.49" y1="50.8" x2="116.84" y2="50.8" width="0.1524" layer="91"/>
-<label x="116.84" y="50.8" size="1.778" layer="95" xref="yes"/>
-</segment>
-</net>
 <net name="GND" class="0">
 <segment>
@@
 <label x="166.37" y="81.28" size="1.778" layer="95" xref="yes"/>
 </segment>
+<segment>
+<pinref part="IC1" gate="G$1" pin="RC6/TX/CK"/>
+<wire x1="102.87" y1="57.15" x2="110.49" y2="57.15" width="0.1524" layer="91"/>
+<wire x1="110.49" y1="57.15" x2="110.49" y2="50.8" width="0.1524" layer="91"/>
+<wire x1="110.49" y1="50.8" x2="116.84" y2="50.8" width="0.1524" layer="91"/>
+<label x="116.84" y="50.8" size="1.778" layer="95" xref="yes"/>
+</segment>
 </net>
 <net name="RC7" class="0">
@@
 <label x="166.37" y="73.66" size="1.778" layer="95" xref="yes"/>
 </segment>
-</net>
+<segment>
+<pinref part="IC1" gate="G$1" pin="RC7/RX/DT/SDO"/>
+<wire x1="102.87" y1="59.69" x2="111.76" y2="59.69" width="0.1524" layer="91"/>
+<wire x1="111.76" y1="59.69" x2="111.76" y2="54.61" width="0.1524" layer="91"/>
+<wire x1="111.76" y1="54.61" x2="116.84" y2="54.61" width="0.1524" layer="91"/>
+<label x="116.84" y="54.61" size="1.778" layer="95" xref="yes"/>
+</segment>
+</net>

Commit message: Cambios en tarjeta PCB
Connections:
- removed net N$1: IC1.!MCLR!/VPP/RE3
- removed net N$10: IC1.RE2/AN7/OESPP
- removed net N$17: IC1.RC2/CCP1/P1A
- removed net N$8: IC1.RE0/AN5/CK1SPP
- removed net N$9: IC1.RE1/AN6/CK2SPP
- removed net RA3: IC1.RA3/AN3/VREF+, R9.1
- removed net RA4: IC1.RA4/T0CKI/CIOUT/RCV, R10.1
- removed net RA5: IC1.RA5/AN4/!SS!/HLVDIN/C2OUT, R11.1
- removed net RA6: IC1.RA6/OSC2/CLKO, R12.1
- removed net RC0: IC1.RC0/TIOSO/T13CKI, R15.1
- removed net RC1: IC1.RC1/T1OSI/ICCP2/!UOE, R17.1
- new net N1: IC1.VUSB
- new net OUT1: IC1.RE0/AN5/CK1SPP, R9.1
- new net OUT2: IC1.RA5/AN4/!SS!/HLVDIN/C2OUT, R10.1
- new net OUT3: IC1.RA4/T0CKI/CIOUT/RCV, R11.1
- new net OUT4: IC1.RA3/AN3/VREF+, R12.1
- new net OUT5: IC1.RA2/AN2/VREF-/CVREF, R13.1
- new net OUT6: IC1.RA1/AN1, R14.1
- new net OUT7: IC1.RA0/AN0, R15.1
- new net OUT8: IC1.!MCLR!/VPP/RE3, R17.1
- new net T_O: IC1.RC1/T1OSI/ICCP2/!UOE, SV2.3
- new net T_OF: IC1.RC2/CCP1/P1A, SV2.1
- net CLK: now also IC1.RC0/TIOSO/T13CKI; no longer IC1.RA1/AN1
- net DAT: now also IC1.RA6/OSC2/CLKO; no longer IC1.RA2/AN2/VREF-/CVREF
- net RB6: no longer R13.1
- net RB7: no longer R14.1
- net RC6: no longer SV2.3
- net RC7: no longer SV2.1
- net RST: now also IC1.RE2/AN7/OESPP; no longer IC1.RA0/AN0
- net VCC: now also IC1.RE1/AN6/CK2SPP
